Commit message: wheels

File: description/robot_core.xacro (robot description, xacro)
@@ -1,20 +1,52 @@
 <?xml version="1.0"?>
-<robot xmlns:xacro = "https://www.ros.org/wiki/xacro">
-<xacro:include filename="colours.xacro" />
-<link name ="base_link">
-</link>
-<joint name="chassis_joint" type="fixed">
-  <origin xyz="-.1 0 0"/>
+<robot xmlns:xacro="https://www.ros.org/wiki/xacro">
+  <!-- Include external file for color definitions -->
+  <xacro:include filename="colours.xacro" />
+  <!-- Base link of the robot -->
+  <link name="base_link">
+  </link>
+  <!-- Fixed joint connecting the base link to the chassis -->
+  <joint name="chassis_joint" type="fixed">
+    <origin xyz="-.1 0 0"/>
+    <parent link="base_link"/>
+    <child link="chassis"/>
+  </joint>
+  <!-- Chassis link of the robot -->
+  <link name="chassis">
+    <visual>
+      <origin xyz=".15 0 .075"/>
+      <geometry>
+        <box size="0.3 0.3 0.15"/>
+      </geometry>
+      <material name="grey"/>
+    </visual>
+  </link>
+<!-- Left wheel link-->
+<joint name="left_wheel_joint" type="continuous">
   <parent link="base_link"/>
-  <child link="chassis"/>
+  <child link="left_wheel"/>
+  <origin xyz="0 0.175 0" rpy ="-${pi/2} 0 0"/>
+  <axis xyz="0 0 1"/>
 </joint>
-<link name = "chassis">
+<link name="left_wheel">
   <visual>
-  <origin xyz=".15 0 .075"/>
     <geometry>
-      <box size="0.3 0.3 0.15"/>
+      <cylinder radius="0.05" length="0.04"/>
     </geometry>
-    <material name="grey"/>
+    <material name="red"/>
   </visual>
-</link>
+<!-- right wheel link-->
+<joint name="right_wheel_joint" type="continuous">
+  <parent link="base_link"/>
+  <child link="right_wheel"/>
+  <origin xyz="0 -0.175 0" rpy ="${pi/2} 0 0"/>
+  <axis xyz="0 0 -1"/>
+</joint>
+<link name="right_wheel">
+  <visual>
+    <geometry>
+      <cylinder radius="0.05" length="0.04"/>
+    </geometry>
+    <material name="red"/>
+  </visual>
 </robot>

Commit message: rviz first thing done

File: description/robot_core.xacro (robot description, xacro)
@@ -3,4 +3,6 @@
   <!-- Include external file for color definitions -->
   <xacro:include filename="colours.xacro" />
+  <!-- Include the macros file -->
+  <xacro:include filename="inertail_macros.xacro" />
   <!-- Base link of the robot -->
   <link name="base_link">
@@ -21,32 +23,85 @@
       <material name="grey"/>
     </visual>
+    <collision>
+      <origin xyz=".15 0 .075"/>
+      <geometry>
+        <box size="0.3 0.3 0.15"/>
+      </geometry>
+    </collision>
+    <xacro:inertial_box mass="0.5" x="0.3" y="0.3" z="0.15">
+      <origin xyz="0.15 0 0.075"/>
+    </xacro:inertial_box>
   </link>
-<!-- Left wheel link-->
-<joint name="left_wheel_joint" type="continuous">
-  <parent link="base_link"/>
-  <child link="left_wheel"/>
-  <origin xyz="0 0.175 0" rpy ="-${pi/2} 0 0"/>
-  <axis xyz="0 0 1"/>
-</joint>
-<link name="left_wheel">
-  <visual>
-    <geometry>
-      <cylinder radius="0.05" length="0.04"/>
-    </geometry>
-    <material name="red"/>
-  </visual>
-<!-- right wheel link-->
-<joint name="right_wheel_joint" type="continuous">
-  <parent link="base_link"/>
-  <child link="right_wheel"/>
-  <origin xyz="0 -0.175 0" rpy ="${pi/2} 0 0"/>
-  <axis xyz="0 0 -1"/>
-</joint>
-<link name="right_wheel">
-  <visual>
-    <geometry>
-      <cylinder radius="0.05" length="0.04"/>
-    </geometry>
-    <material name="red"/>
-  </visual>
+  <!-- Left wheel joint -->
+  <joint name="left_wheel_joint" type="continuous">
+    <parent link="base_link"/>
+    <child link="left_wheel"/>
+    <origin xyz="0 0.175 0" rpy ="-${pi/2} 0 0"/>
+    <axis xyz="0 0 1"/>
+  </joint>
+  <!-- Left wheel link -->
+  <link name="left_wheel">
+    <visual>
+      <geometry>
+        <cylinder radius="0.05" length="0.04"/>
+      </geometry>
+      <material name="red"/>
+    </visual>
+    <collision>
+      <geometry>
+        <cylinder radius="0.05" length="0.04"/>
+      </geometry>
+    </collision>
+    <xacro:inertial_cylinder mass="0.1" length="0.04" radius="0.05">
+      <origin xyz="0 0 0"/>
+    </xacro:inertial_cylinder>
+  </link>
+  <!-- Right wheel joint -->
+  <joint name="right_wheel_joint" type="continuous">
+    <parent link="base_link"/>
+    <child link="right_wheel"/>
+    <origin xyz="0 -0.175 0" rpy ="${pi/2} 0 0"/>
+    <axis xyz="0 0 -1"/>
+  </joint>
+  <!-- Right wheel link -->
+  <link name="right_wheel">
+    <visual>
+      <geometry>
+        <cylinder radius="0.05" length="0.04"/>
+      </geometry>
+      <material name="red"/>
+    </visual>
+    <collision>
+      <geometry>
+        <cylinder radius="0.05" length="0.04"/>
+      </geometry>
+    </collision>
+    <xacro:inertial_cylinder mass="0.1" length="0.04" radius="0.05">
+      <origin xyz="0 0 0"/>
+    </xacro:inertial_cylinder>
+  </link>
+  <!-- Front wheel joint -->
+  <joint name="front_wheel_joint" type="fixed">
+    <parent link="chassis"/>
+    <child link="front_wheel"/>
+    <origin xyz="0.24 0 0"/>
+    <axis xyz="0 1 0"/>
+  </joint>
+  <!-- Front wheel link -->
+  <link name="front_wheel">
+    <visual>
+      <geometry>
+        <sphere radius="0.05"/>
+      </geometry>
+      <material name="blue"/>
+    </visual>
+    <collision>
+      <geometry>
+        <sphere radius="0.05"/>
+      </geometry>
+    </collision>
+    <xacro:inertial_sphere mass="0.5" radius="0.05">
+      <origin xyz="0 0 0"/>
+    </xacro:inertial_sphere>
+  </link>
 </robot>
