Commit message: finished

File: description/robot.urdf.xacro (robot description, xacro)
@@ -3,3 +3,4 @@
     <!-- link to robot core-->
     <xacro:include filename="robot_core.xacro" />
+    <xacro:include filename="gazebo_control.xacro" />
 </robot>

File: description/robot_core.xacro (robot description, xacro)
@@ -33,4 +33,7 @@
     </xacro:inertial_box>
   </link>
+  <gazebo refrence="chassis">
+    <material> Gazebo/White</material>
+    </gazebo>
   <!-- Left wheel joint -->
   <joint name="left_wheel_joint" type="continuous">
@@ -57,4 +60,7 @@
     </xacro:inertial_cylinder>
   </link>
+  <gazebo refrence="left_wheel">
+    <material> Gazebo/Red</material>
+    </gazebo>
   <!-- Right wheel joint -->
   <joint name="right_wheel_joint" type="continuous">
@@ -81,4 +87,7 @@
     </xacro:inertial_cylinder>
   </link>
+<gazebo refrence="right_wheel">
+    <material> Gazebo/Red</material>
+    </gazebo>
   <!-- Front wheel joint -->
   <joint name="front_wheel_joint" type="fixed">
@@ -105,3 +114,6 @@
     </xacro:inertial_sphere>
   </link>
+  <gazebo refrence="front_wheel">
+    <material> Gazebo/Blue</material>
+    </gazebo>
 </robot>
